File: Main_PCB_V2/MRIRobot_PCB.kicad_sch (KiCad schematic)
At the start: 197 parts, among them J1 Conn_01x05, J10 Homing, J11 Homing, J12 Homing, J13 Homing, J14 Homing, J15 Homing, J16 Homing, J17 Conn_01x08, J18 Conn_01x08, J19 Conn_01x08, J2 Conn_01x05, J20 Conn_01x08, J21 Conn_01x08, J22 Conn_01x03, J23 Conn_01x03, J24 Conn_01x08, J25 Conn_01x03, J26 Conn_01x03, J27 Conn_01x08, J3 Conn_01x05, J4 USB_C_Receptacle_USB2.0_16P, J5 Conn_01x05, J6 Conn_01x05, J7 Conn_01x05, J8 Conn_01x05, J9 Power In, SW5 Toggle_Switch2, SW6 Toggle_Switch3, U1 NUCLEO-F446RE, U2 FT231XS, U3 CMOD_A7_FPGA, U4 LM22676MR-5, U5 LM22676MR-ADJ

Commit message: finished new PCB and ordered
Parts:
- added D100, D101, D102, D103, D104, D105, D106, D107, D108, D88, D89, D90, D91, D92, D93, D94, D95, D96, D97, D98, D99: D_TVS, Diode_SMD:D_SOD-123F, symbol Device:D_TVS
- added D109: D, Diode_SMD:D_SMA_Handsoldering, symbol Device:D
- added H7, H8, H9: MountingHole, MountingHole:MountingHole_3.2mm_M3, symbol Mechanical:MountingHole
- added J28, J29, J30, J31: RJ45_RB1-125B8G1A, Connector_RJ:RJ45_UDE_RB1-125B8G1A, symbol Connector:RJ45_RB1-125B8G1A
- added Q1: SUD08P06-155L, Package_TO_SOT_SMD:TO-252-2, symbol Transistor_FET:SUD08P06-155L
- added R6: 100K, Resistor_SMD:R_0805_2012Metric, symbol Device:R
- U1: footprint STM32:MODULE_NUCLEO-F446RE -> NUCLEO-F446RE:MODULE_NUCLEO-F446RE
- U6, U7, U8: value ~ -> LSF0108
Connections:
- net +24V: now also D109.1 (K), Q1.3 (S); no longer J9.2 (Pin_2)
- net 5V_E: now also J28.R5 (TD2-), J29.R5 (TD2-), J30.R5 (TD2-), J31.R9 (TD4-)
- net A0: now also D90.1 (A1), J28.R4 (TD2+)
- net A1: now also D91.1 (A1), J28.R8 (TD4+)
- net A2: now also D96.1 (A1), J29.R4 (TD2+)
- net A3: now also D97.1 (A1), J29.R8 (TD4+)
- net A4: now also D102.1 (A1), J30.R4 (TD2+)
- net A5: now also D103.1 (A1), J30.R8 (TD4+)
- net A6: now also D107.1 (A1), J31.R5 (TD2-)
- net B0: now also D88.1 (A1), J28.R2 (TD1+)
- net B1: now also D89.1 (A1), J28.R6 (TD3+)
- net B2: now also D94.1 (A1), J29.R2 (TD1+)
- net B3: now also D95.1 (A1), J29.R6 (TD3+)
- net B4: now also D100.1 (A1), J30.R2 (TD1+)
- net B5: now also D101.1 (A1), J30.R6 (TD3+)
- net B6: now also D106.1 (A1), J31.R3 (TD1-)
- net GND: now also D100.2 (A2), D101.2 (A2), D102.2 (A2), D103.2 (A2), D104.2 (A2), D105.2 (A2), D106.2 (A2), D107.2 (A2), D108.2 (A2), D88.2 (A2), D89.2 (A2), D90.2 (A2), D91.2 (A2), D92.2 (A2), D93.2 (A2), D94.2 (A2), D95.2 (A2), D96.2 (A2), D97.2 (A2), D98.2 (A2), D99.2 (A2), J28.R9 (TD4-), J28.SH, J29.R9 (TD4-), J29.SH, J30.R9 (TD4-), J30.SH, J31.R2 (TD1+), J31.R4 (TD2+), J31.R6 (TD3+), J31.R8 (TD4+), J31.SH, R6.2
- net I0: now also D92.1 (A1), J28.R3 (TD1-)
- net I1: now also D93.1 (A1), J28.R7 (TD3-)
- net I2: now also D98.1 (A1), J29.R3 (TD1-)
- net I3: now also D99.1 (A1), J29.R7 (TD3-)
- net I4: now also D104.1 (A1), J30.R3 (TD1-)
- net I5: now also D105.1 (A1), J30.R7 (TD3-)
- net I6: now also D108.1 (A1), J31.R7 (TD3-)
- new net: D109.2 (A), Q1.1 (G), R6.1
- new net: J9.2 (Pin_2), Q1.2 (D)
- no-connect marks 68 -> 92
Other:
- moved on the sheet: C1, C17, C18, C19, D1, D12, D13, D14, D17, D19, D20, D21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
