File: Motor_Adapt_C/Motor_Adapt_C.kicad_pcb (KiCad board)
At the start: 2 copper layers, 34.5 x 36.8 mm, 12 parts, among them J1 Conn_01x08, J2 RJCSE538001, J3 Conn_01x03

Commit message: updated pcbs
Parts:
- added D1: D_TVS, Diode_SMD:D_SOD-123F, F.Cu at (45.8, 64.5)
- added D2: D_TVS, Diode_SMD:D_SOD-123F, F.Cu at (50.2, 64.5)
- added D3: D_TVS, Diode_SMD:D_SOD-123F, F.Cu at (53.8, 64.5)
- added H1: MountingHole, MountingHole:MountingHole_3.2mm_M3, F.Cu at (58.0, 74.0)
- added H2: MountingHole, MountingHole:MountingHole_3.2mm_M3, F.Cu at (33.5, 74.0)
- moved J1 4.03 mm to (36.5, 81.5)
- moved C1 3.76 mm to (52.5, 71.7)
- moved C2 3.76 mm to (48.5, 71.7)
- moved C3 3.76 mm to (44.5, 71.7)
- moved R2 3.76 mm to (47.5, 68.7)
- moved R1 3.76 mm to (51.5, 68.8)
- moved R3 3.76 mm to (43.5, 68.8)
- moved U1 3.47 mm to (52.5, 76.3)
- moved U2 3.47 mm to (48.7, 76.3)
- moved U3 3.47 mm to (44.8, 76.4)
Routing:
- net GND: track 16.4 -> 26.2 mm, vias 21 -> 36
- net /C_B: track 6.59 -> 11.7 mm
- net /C_I: track 5.08 -> 9.93 mm
- net /C_A: track 8.61 -> 12.9 mm
- net /Cos: track 26.2 -> 30.4 mm
- net /Sin: track 25.8 -> 30.0 mm
- net /MC_B: track 4.59 -> 6.28 mm
- net /MC_I: track 4.08 -> 5.03 mm
- net /MC_A: track 6.50 -> 7.45 mm
Other:
- board size 34.5 x 36.8 mm -> 34.5 x 41 mm
