File: Motor_Adapt_C/Motor_Adapt_C.kicad_sch (KiCad schematic)
At the start: 12 parts, among them J1 Conn_01x08, J2 RJCSE538001, J3 Conn_01x03

Commit message: updated pcbs
Parts:
- added D1, D2, D3: D_TVS, Diode_SMD:D_SOD-123F, symbol Device:D_TVS
- added H1, H2: MountingHole, MountingHole:MountingHole_3.2mm_M3, symbol Mechanical:MountingHole
Connections:
- net C_A: now also D1.1 (A1)
- net C_B: now also D2.1 (A1)
- net C_I: now also D3.1 (A1)
- net GND: now also D1.2 (A2), D2.2 (A2), D3.2 (A2)
Other:
- note added: "TVS Diodes"
