File: Motor_Adapt_M/Motor_Adapt_M.kicad_pcb (KiCad board)
At the start: 2 copper layers, 34.8 x 24.5 mm, 3 parts, among them J1 Conn_01x08, J2 RJCSE538001, J3 Conn_01x03

Commit message: updated pcbs
Parts:
- removed J2: RJCSE538001, RJCSE538001:AMPHENOL_RJCSE538001
- added H1: MountingHole, MountingHole:MountingHole_3.2mm_M3, F.Cu at (61.0, 57.5)
- added H2: MountingHole, MountingHole:MountingHole_3.2mm_M3, F.Cu at (36.5, 57.5)
- added J4: 54602-908LF, ethernet_54602-908LF:ethernet_54602-908LF, F.Cu at (59.7, 48.6)
- moved J1 8.04 mm to (40.0, 63.5)
Routing:
- net +5V: track 7.25 -> 21.7 mm
- net /C_I: track 5.18 -> 18.7 mm
- net GND: track 12.3 -> 0.00 mm, vias 20 -> 23
- net /C_B: track 5.20 -> 16.8 mm
- net /Sin: track 14.6 -> 23.3 mm
- net /Cos: track 14.3 -> 22.6 mm
- net /C_A: track 5.39 -> 12.8 mm
Other:
- board size 34.8 x 24.5 mm -> 34.5 x 32.5 mm

Commit message: update
Connections:
- J4 pad 1: /C_B -> +5V
- J4 pad 2: +5V -> GND
- J4 pad 3: GND -> /C_A
- J4 pad 5: /C_I -> /C_B
- J4 pad 6: /C_A -> GND
- J4 pad 7: GND -> /C_I
Routing:
- net /C_A: track 12.8 -> 21.6 mm
- net +5V: track 21.7 -> 29.3 mm
- net /C_I: track 18.7 -> 17.2 mm
- net /C_B: track 16.8 -> 15.7 mm
- net /Sin: track 23.3 -> 22.2 mm
Changed lines of the file:
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@@
 			(layers "*.Cu" "*.Mask")
 			(remove_unused_layers no)
-			(net 5 "/C_B")
+			(net 4 "+5V")
 			(pinfunction "1")
 			(pintype "unspecified")
@@
 			(layers "*.Cu" "*.Mask")
 			(remove_unused_layers no)
-			(net 4 "+5V")
+			(net 1 "GND")
 			(pinfunction "2")
 			(pintype "unspecified")
@@
 			(layers "*.Cu" "*.Mask")
 			(remove_unused_layers no)
-			(net 1 "GND")
+			(net 7 "/C_A")
 			(pinfunction "3")
 			(pintype "unspecified")
@@
 			(layers "*.Cu" "*.Mask")
 			(remove_unused_layers no)
-			(net 6 "/C_I")
+			(net 5 "/C_B")
 			(pinfunction "5")
 			(pintype "unspecified")
@@
 			(layers "*.Cu" "*.Mask")
 			(remove_unused_layers no)
-			(net 7 "/C_A")
+			(net 1 "GND")
 			(pinfunction "6")
 			(pintype "unspecified")
@@
 			(layers "*.Cu" "*.Mask")
 			(remove_unused_layers no)
-			(net 1 "GND")
+			(net 6 "/C_I")
 			(pinfunction "7")
 			(pintype "unspecified")
@@
 	)
 	(via
+		(at 43.5 57)
+		(size 0.6)
+		(drill 0.3)
+		(layers "F.Cu" "B.Cu")
+		(free yes)
+		(net 1)
+	)
+	(via
 		(at 39.25 52.5)
 		(size 0.6)
@@
 	)
 	(via
+		(at 49.25 55)
+		(size 0.6)
+		(drill 0.3)
+		(layers "F.Cu" "B.Cu")
+		(free yes)
+		(net 1)
+	)
+	(via
 		(at 34.5 38.5)
 		(size 0.6)
@@
 	)
 	(via
-		(at 43 52.75)
-		(size 0.6)
-		(drill 0.3)
-		(layers "F.Cu" "B.Cu")
-		(free yes)
-		(net 1)
-	)
-	(via
-		(at 50.75 53)
-		(size 0.6)
-		(drill 0.3)
-		(layers "F.Cu" "B.Cu")
-		(free yes)
-		(net 1)
-	)
-	(via
-		(at 48.75 49.25)
+		(at 43.5 53.75)
+		(size 0.6)
+		(drill 0.3)
+		(layers "F.Cu" "B.Cu")
+		(free yes)
+		(net 1)
+	)
+	(via
+		(at 50.25 53.5)
 		(size 0.6)
 		(drill 0.3)
@@
 	)
 	(via
-		(at 47.75 54.5)
-		(size 0.6)
-		(drill 0.3)
-		(layers "F.Cu" "B.Cu")
-		(free yes)
-		(net 1)
-	)
-	(via
-		(at 55.25 53.5)
-		(size 0.6)
-		(drill 0.3)
-		(layers "F.Cu" "B.Cu")
-		(free yes)
+		(at 49.75 59.75)
+		(size 0.6)
+		(drill 0.3)
+		(layers "F.Cu" "B.Cu")
+		(free yes)
+		(net 1)
+	)
+	(segment
+		(start 53.25 51.2)
+		(end 53.31 51.14)
+		(width 0.5)
+		(layer "B.Cu")
 		(net 1)
 	)
@@
 	)
 	(segment
-		(start 42 61.5)
+		(start 40.75 62.75)
 		(end 40 63.5)
 		(width 0.5)
@@
 	)
 	(segment
-		(start 42 51.615)
-		(end 42 61.5)
+		(start 40.75 50.365)
+		(end 40.75 62.75)
 		(width 0.5)
 		(layer "F.Cu")
@@
 	(segment
 		(start 34.54 44.155)
-		(end 42 51.615)
+		(end 40.75 50.365)
 		(width 0.5)
 		(layer "F.Cu")
@@
 	)
 	(segment
+		(start 47.5 58.5)
+		(end 47 58)
+		(width 0.5)
+		(layer "F.Cu")
+		(net 4)
+	)
+	(segment
+		(start 51.189339 45.75)
+		(end 56.81 45.75)
+		(width 0.5)
+		(layer "F.Cu")
+		(net 4)
+	)
+	(segment
+		(start 56.81 45.75)
+		(end 59.66 48.6)
+		(width 0.5)
+		(layer "F.Cu")
+		(net 4)
+	)
+	(segment
+		(start 47 58)
+		(end 47 49.939339)
+		(width 0.5)
+		(layer "F.Cu")
+		(net 4)
+	)
+	(segment
+		(start 47 49.939339)
+		(end 51.189339 45.75)
+		(width 0.5)
+		(layer "F.Cu")
+		(net 4)
+	)
+	(segment
 		(start 47.5 63.5)
-		(end 47.5 58.25)
+		(end 47.5 58.5)
 		(width 0.5)
 		(layer "F.Cu")
@@
 	)
 	(segment
-		(start 57.25 50)
-		(end 58.39 51.14)
-		(width 0.5)
-		(layer "F.Cu")
-		(net 4)
-	)
-	(segment
-		(start 52.225 50.690578)
-		(end 52.915578 50)
-		(width 0.5)
-		(layer "F.Cu")
-		(net 4)
-	)
-	(segment
-		(start 47.5 58.25)
-		(end 52.225 53.525)
-		(width 0.5)
-		(layer "F.Cu")
-		(net 4)
-	)
-	(segment
-		(start 52.225 53.525)
-		(end 52.225 50.690578)
-		(width 0.5)
-		(layer "F.Cu")
-		(net 4)
-	)
-	(segment
-		(start 52.915578 50)
-		(end 57.25 50)
-		(width 0.5)
-		(layer "F.Cu")
-		(net 4)
-	)
-	(segment
-		(start 59.66 48.6)
-		(end 59.66 51.404422)
+		(start 54.5 48.68)
+		(end 54.58 48.6)
+		(width 0.5)
+		(layer "F.Cu")
+		(net 5)
+	)
+	(segment
+		(start 54.5 55.564422)
+		(end 54.5 48.68)
 		(width 0.5)
 		(layer "F.Cu")
@@
 	)
 	(segment
-		(start 59.66 51.404422)
-		(end 55 56.064422)
+		(start 55 56.064422)
+		(end 54.5 55.564422)
 		(width 0.5)
 		(layer "F.Cu")
@@
 	)
 	(segment
-		(start 54.315578 48.6)
-		(end 52 50.915578)
+		(start 54.58 48.6)
+		(end 54.315578 48.6)
+		(width 0.5)
+		(layer "B.Cu")
+		(net 5)
+	)
+	(segment
+		(start 54.85 48.6)
+		(end 54.58 48.6)
+		(width 0.5)
+		(layer "B.Cu")
+		(net 5)
+	)
+	(segment
+		(start 57.5 63.5)
+		(end 52.04 58.04)
 		(width 0.5)
 		(layer "B.Cu")
@@
 	)
 	(segment
-		(start 52 50.915578)
-		(end 52 58)
+		(start 52.04 58.04)
+		(end 52.04 48.6)
 		(width 0.5)
 		(layer "B.Cu")
@@
 	)
 	(segment
-		(start 54.58 48.6)
-		(end 54.315578 48.6)
-		(width 0.5)
-		(layer "B.Cu")
-		(net 6)
+		(start 52.5 63.5)
+		(end 52.5 58.5)
+		(width 0.5)
+		(layer "F.Cu")
+		(net 7)
+	)
+	(segment
+		(start 53.25 49.2475)
+		(end 53.25 47.5)
+		(width 0.5)
+		(layer "F.Cu")
+		(net 7)
+	)
+	(segment
+		(start 53.25 47.5)
+		(end 53.75 47)
+		(width 0.5)
+		(layer "F.Cu")
+		(net 7)
+	)
+	(segment
+		(start 55.76 47)
+		(end 57.12 48.36)
+		(width 0.5)
+		(layer "F.Cu")
+		(net 7)
+	)
+	(segment
+		(start 52.5 58.5)
+		(end 52 58)
+		(width 0.5)
+		(layer "F.Cu")
+		(net 7)
 	)
 	(segment
 		(start 52 58)
-		(end 57.5 63.5)
-		(width 0.5)
-		(layer "B.Cu")
-		(net 6)
-	)
-	(segment
-		(start 54.85 48.6)
-		(end 54.58 48.6)
-		(width 0.5)
-		(layer "B.Cu")
-		(net 6)
-	)
-	(segment
-		(start 53.31 51.14)
-		(end 53.31 57.69)
+		(end 52 50.4975)
 		(width 0.5)
 		(layer "F.Cu")
@@
 	)
 	(segment
-		(start 52.5 58.5)
-		(end 52.5 63.5)
+		(start 53.75 47)
+		(end 55.76 47)
 		(width 0.5)
 		(layer "F.Cu")
@@
 	)
 	(segment
-		(start 53.31 57.69)
-		(end 52.5 58.5)
+		(start 57.12 48.36)
+		(end 57.12 48.6)
 		(width 0.5)
 		(layer "F.Cu")
@@
 	)
 	(segment
-		(start 53.25 51.2)
-		(end 53.31 51.14)
-		(width 0.5)
-		(layer "B.Cu")
+		(start 52 50.4975)
+		(end 53.25 49.2475)
+		(width 0.5)
+		(layer "F.Cu")
 		(net 7)
 	)
