File: Power_PCB_V2/Power_PCB.kicad_pcb (KiCad board)
At the start: 2 copper layers, 142 x 45 mm, 61 parts, among them J1 PWR IN, J10 Motor, J2 PWR MB, J3 Conn_01x03, J4 Motor, J5 Motor, J6 Motor, J7 Motor, J8 Motor, J9 Motor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

Commit message: updated PCBs
Parts:
- added R13: 2.5k, Resistor_SMD:R_0805_2012Metric, B.Cu at (107.8, 66.0)
Routing:
- net /Relay_in: track 9.19 -> 12.5 mm
- net GND: track 11.1 -> 12.5 mm, vias 97 -> 98

Commit message: updated pcbs
Changed lines of the file:
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@@
 		(layer "F.Cu")
 		(at 49 48 90)
-		(descr "Connector XT30 Vertical Cable Male, https://www.tme.eu/en/Document/3cbfa5cfa544d79584972dd5234a409e/XT30U%20SPEC.pdf")
+		(descr "Connector XT30 Vertical Cable Male, https://www.tme.eu/Document/7d9d972ae3468777f69ec2ee99897652/XT30U-M.pdf")
 		(tags "RC Connector XT30")
 		(property "Reference" "J7"
@@
 			)
 		)
-		(pad "1" thru_hole rect
+		(pad "1" thru_hole roundrect
 			(at 0 0 90)
 			(size 3.8 3.8)
@@
 			(layers "*.Cu" "*.Mask")
 			(remove_unused_layers no)
+			(roundrect_rratio 0.2)
 			(net 24 "/24V_M1")
 			(pinfunction "Pin_1")
@@
 		(pad "1" thru_hole circle
 			(at 0 1.55)
-			(size 1.524 1.524)
-			(drill 0.762)
+			(size 2.54 2.54)
+			(drill 1.3)
 			(layers "*.Cu" "*.Mask")
 			(remove_unused_layers no)
@@
 		(pad "2" thru_hole circle
 			(at 0 6.35)
-			(size 1.524 1.524)
-			(drill 0.762)
+			(size 2.54 2.54)
+			(drill 1.3)
 			(layers "*.Cu" "*.Mask")
 			(remove_unused_layers no)
@@
 		(pad "3" thru_hole circle
 			(at 0 11)
-			(size 1.524 1.524)
-			(drill 0.762)
+			(size 2.54 2.54)
+			(drill 1.3)
 			(layers "*.Cu" "*.Mask")
 			(remove_unused_layers no)
@@
 		(layer "F.Cu")
 		(at 58 48 90)
-		(descr "Connector XT30 Vertical Cable Male, https://www.tme.eu/en/Document/3cbfa5cfa544d79584972dd5234a409e/XT30U%20SPEC.pdf")
+		(descr "Connector XT30 Vertical Cable Male, https://www.tme.eu/Document/7d9d972ae3468777f69ec2ee99897652/XT30U-M.pdf")
 		(tags "RC Connector XT30")
 		(property "Reference" "J9"
@@
 			(layer "F.Fab")
 		)
-		(fp_text user "-"
-			(at -4 0 90)
+		(fp_text user "+"
+			(at 9 0 90)
 			(layer "F.SilkS")
 			(effects
@@
 			)
 		)
-		(fp_text user "+"
-			(at 9 0 90)
+		(fp_text user "-"
+			(at -4 0 90)
 			(layer "F.SilkS")
 			(effects
@@
 			)
 		)
-		(pad "1" thru_hole rect
+		(pad "1" thru_hole roundrect
 			(at 0 0 90)
 			(size 3.8 3.8)
@@
 			(layers "*.Cu" "*.Mask")
 			(remove_unused_layers no)
+			(roundrect_rratio 0.2)
 			(net 31 "/24V_M2")
 			(pinfunction "Pin_1")
@@
 		(pad "1" thru_hole circle
 			(at 0 1.55)
-			(size 1.524 1.524)
-			(drill 0.762)
+			(size 2.54 2.54)
+			(drill 1.3)
 			(layers "*.Cu" "*.Mask")
 			(remove_unused_layers no)
@@
 		(pad "2" thru_hole circle
 			(at 0 6.35)
-			(size 1.524 1.524)
-			(drill 0.762)
+			(size 2.54 2.54)
+			(drill 1.3)
 			(layers "*.Cu" "*.Mask")
 			(remove_unused_layers no)
@@
 		(pad "3" thru_hole circle
 			(at 0 11)
-			(size 1.524 1.524)
-			(drill 0.762)
+			(size 2.54 2.54)
+			(drill 1.3)
 			(layers "*.Cu" "*.Mask")
 			(remove_unused_layers no)
@@
 		(pad "1" thru_hole circle
 			(at 0 1.55)
-			(size 1.524 1.524)
-			(drill 0.762)
+			(size 2.54 2.54)
+			(drill 1.3)
 			(layers "*.Cu" "*.Mask")
 			(remove_unused_layers no)
@@
 		(pad "2" thru_hole circle
 			(at 0 6.35)
-			(size 1.524 1.524)
-			(drill 0.762)
+			(size 2.54 2.54)
+			(drill 1.3)
 			(layers "*.Cu" "*.Mask")
 			(remove_unused_layers no)
@@
 		(pad "3" thru_hole circle
 			(at 0 11)
-			(size 1.524 1.524)
-			(drill 0.762)
+			(size 2.54 2.54)
+			(drill 1.3)
 			(layers "*.Cu" "*.Mask")
 			(remove_unused_layers no)
@@
 		(layer "F.Cu")
 		(at 76 48 90)
-		(descr "Connector XT30 Vertical Cable Male, https://www.tme.eu/en/Document/3cbfa5cfa544d79584972dd5234a409e/XT30U%20SPEC.pdf")
+		(descr "Connector XT30 Vertical Cable Male, https://www.tme.eu/Document/7d9d972ae3468777f69ec2ee99897652/XT30U-M.pdf")
 		(tags "RC Connector XT30")
 		(property "Reference" "J8"
@@
 			(layer "F.Fab")
 		)
-		(fp_text user "-"
-			(at -4 0 90)
+		(fp_text user "+"
+			(at 9 0 90)
 			(layer "F.SilkS")
 			(effects
@@
 			)
 		)
-		(fp_text user "+"
-			(at 9 0 90)
+		(fp_text user "-"
+			(at -4 0 90)
 			(layer "F.SilkS")
 			(effects
@@
 			)
 		)
-		(pad "1" thru_hole rect
+		(pad "1" thru_hole roundrect
 			(at 0 0 90)
 			(size 3.8 3.8)
@@
 			(layers "*.Cu" "*.Mask")
 			(remove_unused_layers no)
+			(roundrect_rratio 0.2)
 			(net 27 "/24V_M4")
 			(pinfunction "Pin_1")
@@
 		(pad "1" thru_hole circle
 			(at 0 1.55)
-			(size 1.524 1.524)
-			(drill 0.762)
+			(size 2.54 2.54)
+			(drill 1.3)
 			(layers "*.Cu" "*.Mask")
 			(remove_unused_layers no)
@@
 		(pad "2" thru_hole circle
 			(at 0 6.35)
-			(size 1.524 1.524)
-			(drill 0.762)
+			(size 2.54 2.54)
+			(drill 1.3)
 			(layers "*.Cu" "*.Mask")
 			(remove_unused_layers no)
@@
 		(pad "3" thru_hole circle
 			(at 0 11)
-			(size 1.524 1.524)
-			(drill 0.762)
+			(size 2.54 2.54)
+			(drill 1.3)
 			(layers "*.Cu" "*.Mask")
 			(remove_unused_layers no)
@@
 		(layer "F.Cu")
 		(at 67 48 90)
-		(descr "Connector XT30 Vertical Cable Male, https://www.tme.eu/en/Document/3cbfa5cfa544d79584972dd5234a409e/XT30U%20SPEC.pdf")
+		(descr "Connector XT30 Vertical Cable Male, https://www.tme.eu/Document/7d9d972ae3468777f69ec2ee99897652/XT30U-M.pdf")
 		(tags "RC Connector XT30")
 		(property "Reference" "J5"
@@
 			(layer "F.Fab")
 		)
-		(fp_text user "-"
-			(at -4 0 90)
+		(fp_text user "+"
+			(at 9 0 90)
 			(layer "F.SilkS")
 			(effects
@@
 			)
 		)
-		(fp_text user "+"
-			(at 9 0 90)
+		(fp_text user "-"
+			(at -4 0 90)
 			(layer "F.SilkS")
 			(effects
@@
 			)
 		)
-		(pad "1" thru_hole rect
+		(pad "1" thru_hole roundrect
 			(at 0 0 90)
 			(size 3.8 3.8)
@@
 			(layers "*.Cu" "*.Mask")
 			(remove_unused_layers no)
+			(roundrect_rratio 0.2)
 			(net 20 "/24V_M3")
 			(pinfunction "Pin_1")
@@
 		(pad "1" thru_hole circle
 			(at 0 1.55)
-			(size 1.524 1.524)
-			(drill 0.762)
+			(size 2.54 2.54)
+			(drill 1.3)
 			(layers "*.Cu" "*.Mask")
 			(remove_unused_layers no)
@@
 		(pad "2" thru_hole circle
 			(at 0 6.35)
-			(size 1.524 1.524)
-			(drill 0.762)
+			(size 2.54 2.54)
+			(drill 1.3)
 			(layers "*.Cu" "*.Mask")
 			(remove_unused_layers no)
@@
 		(pad "3" thru_hole circle
 			(at 0 11)
-			(size 1.524 1.524)
-			(drill 0.762)
+			(size 2.54 2.54)
+			(drill 1.3)
 			(layers "*.Cu" "*.Mask")
 			(remove_unused_layers no)
@@
 		(layer "F.Cu")
 		(at 94 48 90)
-		(descr "Connector XT30 Vertical Cable Male, https://www.tme.eu/en/Document/3cbfa5cfa544d79584972dd5234a409e/XT30U%20SPEC.pdf")
+		(descr "Connector XT30 Vertical Cable Male, https://www.tme.eu/Document/7d9d972ae3468777f69ec2ee99897652/XT30U-M.pdf")
 		(tags "RC Connector XT30")
 		(property "Reference" "J6"
@@
 			)
 		)
-		(pad "1" thru_hole rect
+		(pad "1" thru_hole roundrect
 			(at 0 0 90)
 			(size 3.8 3.8)
@@
 			(layers "*.Cu" "*.Mask")
 			(remove_unused_layers no)
+			(roundrect_rratio 0.2)
 			(net 19 "/24V_M6")
 			(pinfunction "Pin_1")
@@
 		(layer "F.Cu")
 		(at 40 48.25 90)
-		(descr "Connector XT30 Vertical Cable Male, https://www.tme.eu/en/Document/3cbfa5cfa544d79584972dd5234a409e/XT30U%20SPEC.pdf")
+		(descr "Connector XT30 Vertical Cable Male, https://www.tme.eu/Document/7d9d972ae3468777f69ec2ee99897652/XT30U-M.pdf")
 		(tags "RC Connector XT30")
 		(property "Reference" "J4"
@@
 			)
 		)
-		(pad "1" thru_hole rect
+		(pad "1" thru_hole roundrect
 			(at 0 0 90)
 			(size 3.8 3.8)
@@
 			(layers "*.Cu" "*.Mask")
 			(remove_unused_layers no)
+			(roundrect_rratio 0.2)
 			(net 22 "/24V_M0")
 			(pinfunction "Pin_1")
@@
 		(pad "1" thru_hole circle
 			(at 0 1.55)
-			(size 1.524 1.524)
-			(drill 0.762)
+			(size 2.54 2.54)
+			(drill 1.3)
 			(layers "*.Cu" "*.Mask")
 			(remove_unused_layers no)
@@
 		(pad "2" thru_hole circle
 			(at 0 6.35)
-			(size 1.524 1.524)
-			(drill 0.762)
+			(size 2.54 2.54)
+			(drill 1.3)
 			(layers "*.Cu" "*.Mask")
 			(remove_unused_layers no)
@@
 		(pad "3" thru_hole circle
 			(at 0 11)
-			(size 1.524 1.524)
-			(drill 0.762)
+			(size 2.54 2.54)
+			(drill 1.3)
 			(layers "*.Cu" "*.Mask")
 			(remove_unused_layers no)
@@
 		(layer "F.Cu")
 		(at 85 48 90)
-		(descr "Connector XT30 Vertical Cable Male, https://www.tme.eu/en/Document/3cbfa5cfa544d79584972dd5234a409e/XT30U%20SPEC.pdf")
+		(descr "Connector XT30 Vertical Cable Male, https://www.tme.eu/Document/7d9d972ae3468777f69ec2ee99897652/XT30U-M.pdf")
 		(tags "RC Connector XT30")
 		(property "Reference" "J10"
@@
 			(layer "F.Fab")
 		)
-		(fp_text user "-"
-			(at -4 0 90)
+		(fp_text user "+"
+			(at 9 0 90)
 			(layer "F.SilkS")
 			(effects
@@
 			)
 		)
-		(fp_text user "+"
-			(at 9 0 90)
+		(fp_text user "-"
+			(at -4 0 90)
 			(layer "F.SilkS")
 			(effects
@@
 			)
 		)
-		(pad "1" thru_hole rect
+		(pad "1" thru_hole roundrect
 			(at 0 0 90)
 			(size 3.8 3.8)
@@
 			(layers "*.Cu" "*.Mask")
 			(remove_unused_layers no)
+			(roundrect_rratio 0.2)
 			(net 29 "/24V_M5")
 			(pinfunction "Pin_1")
@@
 		(pad "1" thru_hole circle
 			(at 0 1.55)
-			(size 1.524 1.524)
-			(drill 0.762)
+			(size 2.54 2.54)
+			(drill 1.3)
 			(layers "*.Cu" "*.Mask")
 			(remove_unused_layers no)
@@
 		(pad "2" thru_hole circle
 			(at 0 6.35)
-			(size 1.524 1.524)
-			(drill 0.762)
+			(size 2.54 2.54)
+			(drill 1.3)
 			(layers "*.Cu" "*.Mask")
 			(remove_unused_layers no)
@@
 		(pad "3" thru_hole circle
 			(at 0 11)
-			(size 1.524 1.524)
-			(drill 0.762)
+			(size 2.54 2.54)
+			(drill 1.3)
 			(layers "*.Cu" "*.Mask")
 			(remove_unused_layers no)
@@
 		(tags "resistor")
 		(property "Reference" "R13"
-			(at 0 1.65 360)
+			(at 0 1.65 0)
 			(layer "B.SilkS")
 			(effects
@@
 		)
 		(property "Value" "2.5k"
-			(at 0 -1.65 360)
+			(at 0 -1.65 0)
 			(layer "B.Fab")
 			(effects
@@
 		)
 		(fp_text user "${REFERENCE}"
-			(at 0 0 360)
+			(at 0 0 0)
 			(layer "B.Fab")
 			(effects
@@
 		(fp_poly
 			(pts
-				(xy -4.73 3.14) (xy -4.97 3.47) (xy -4.49 3.47) (xy -4.73 3.14)
+				(xy -5.04 3.14) (xy -5.38 3.61) (xy -4.7 3.61) (xy -5.04 3.14)
 			)
 			(stroke

Commit message: update
Parts:
- added C3: 220uF, Capacitor_THT:CP_Radial_D8.0mm_P3.50mm, F.Cu at (122.0, 71.3)
- added C4: 220uF, Capacitor_THT:CP_Radial_D8.0mm_P3.50mm, F.Cu at (131.2, 71.5)
Routing:
- net GND: vias 98 -> 96
Other:
- board text added: "CONTROLLER PWR"
- board text removed: "MAIN CONTROLLER PWR"
