File: Power_PCB_V2/Power_PCB.kicad_sch (KiCad schematic)
At the start: 61 parts, among them J1 PWR IN, J10 Motor, J2 PWR MB, J3 Conn_01x03, J4 Motor, J5 Motor, J6 Motor, J7 Motor, J8 Motor, J9 Motor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

Commit message: updated PCBs
Parts:
- added R13: 2.5k, Resistor_SMD:R_0805_2012Metric, symbol Device:R
Connections:
- net GND: now also R13.2
- net Relay_in: now also R13.1
Changed lines of the file:
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@@
 	(wire
 		(pts
+			(xy 165.1 137.16) (xy 165.1 135.89)
+		)
+		(stroke
+			(width 0)
+			(type default)
+		)
+	)
+	(wire
+		(pts
 			(xy 26.67 147.32) (xy 22.86 147.32)
 		)
@@
 	(wire
 		(pts
+			(xy 165.1 147.32) (xy 165.1 144.78)
+		)
+		(stroke
+			(width 0)
+			(type default)
+		)
+	)
+	(wire
+		(pts
 			(xy 213.36 33.02) (xy 215.9 33.02)
 		)
@@
 	(rectangle
 		(start 13.97 121.92)
-		(end 167.64 165.1)
+		(end 180.34 165.1)
 		(stroke
 			(width 0)
@@
 		)
 	)
+	(label "Relay_in"
+		(at 165.1 135.89 0)
+		(fields_autoplaced yes)
+		(effects
+			(font
+				(size 1.27 1.27)
+			)
+			(justify left bottom)
+		)
+	)
 	(label "24V_M5"
 		(at 233.68 66.04 0)
@@
 	)
 	(symbol
+		(lib_id "Device:R")
+		(at 165.1 140.97 0)
+		(unit 1)
+		(exclude_from_sim no)
+		(in_bom yes)
+		(on_board yes)
+		(dnp no)
+		(property "Reference" "R13"
+			(at 167.386 143.51 90)
+			(effects
+				(font
+					(size 1.27 1.27)
+				)
+				(justify left)
+			)
+		)
+		(property "Value" "2.5k"
+			(at 169.926 143.51 90)
+			(effects
+				(font
+					(size 1.27 1.27)
+				)
+				(justify left)
+			)
+		)
+		(property "Footprint" "Resistor_SMD:R_0805_2012Metric"
+			(at 163.322 140.97 90)
+			(effects
+				(font
+					(size 1.27 1.27)
+				)
+				(hide yes)
+			)
+		)
+		(property "Datasheet" "~"
+			(at 165.1 140.97 0)
+			(effects
+				(font
+					(size 1.27 1.27)
+				)
+				(hide yes)
+			)
+		)
+		(property "Description" "Resistor"
+			(at 165.1 140.97 0)
+			(effects
+				(font
+					(size 1.27 1.27)
+				)
+				(hide yes)
+			)
+		)
+		(pin "2"
+		)
+		(pin "1"
+		)
+		(instances
+			(project "Power_PCB"
+				(path "/474d276f-aef6-4d19-92f1-32849a56a83d"
+					(reference "R13")
+					(unit 1)
+				)
+			)
+		)
+	)
+	(symbol
 		(lib_id "Device:Fuse")
 		(at 167.64 66.04 90)
@@
 					(unit 1)
 				)
+			)
+		)
+	)
+	(symbol
+		(lib_id "power:GND")
+		(at 165.1 147.32 0)
+		(unit 1)
+		(exclude_from_sim no)
+		(in_bom yes)
+		(on_board yes)
+		(dnp no)
+		(fields_autoplaced yes)
+		(property "Reference" "#PWR049"
+			(at 165.1 153.67 0)
+			(effects
+				(font
+					(size 1.27 1.27)
+				)
+				(hide yes)
+			)
+		)
+		(property "Value" "GND"
+			(at 165.1 152.4 0)
+			(effects
+				(font
+					(size 1.27 1.27)
+				)
+			)
+		)
+		(property "Footprint" ""
+			(at 165.1 147.32 0)
+			(effects
+				(font
+					(size 1.27 1.27)
+				)
+				(hide yes)
+			)
+		)
+		(property "Datasheet" ""
+			(at 165.1 147.32 0)
+			(effects
+				(font
+					(size 1.27 1.27)
+				)
+				(hide yes)
+			)
+		)
+		(property "Description" "Power symbol creates a global label with name \"GND\" , ground"
+			(at 165.1 147.32 0)
+			(effects
+				(font
+					(size 1.27 1.27)
+				)
+				(hide yes)
+			)
+		)
+		(pin "1"
+		)
+		(instances
+			(project "Power_PCB"
+				(path "/474d276f-aef6-4d19-92f1-32849a56a83d"
+					(reference "#PWR049")
+					(unit 1)
+				)

Commit message: update
Parts:
- added C3, C4: 220uF, Capacitor_THT:CP_Radial_D8.0mm_P3.50mm, symbol Device:C
Connections:
- net +24V: now also C3.1, C4.1
- net GND: now also C3.2, C4.2
