File: Main_PCB_V3/MRIRobot_PCB.kicad_sch (KiCad schematic)
At the start: 335 parts, among them J1 Conn_01x05, J10 Homing, J11 Homing, J12 Homing, J13 Homing, J14 Homing, J15 Homing, J16 Homing, J17 Conn_01x08, J18 Conn_01x08, J19 Conn_01x08, J2 Conn_01x05, J20 Conn_01x08, J21 Conn_01x08, J22 Conn_01x03, J23 Conn_01x03, J24 Conn_01x08, J25 Conn_01x03, J26 Conn_01x03, J27 Conn_01x08, J28 RJCSE538001, J3 Conn_01x05, J32 RJCSE538001, J33 RJCSE538001, J34 RJCSE538001, J4 USB_C_Receptacle_USB2.0_16P, J5 Conn_01x05, J6 Conn_01x05, J7 Conn_01x05, J8 Conn_01x05, J9 Power In, Q1 SUD08P06-155L, SW5 Toggle_Switch2, SW6 Toggle_Switch3, U1 NUCLEO-F446RE, U2 FT231XS, U3 CMOD_A7_FPGA, U4 LM22676MR-5, U5 LM22676MR-ADJ, U6 LSF0108, U7 LSF0108, U8 LSF0108

Commit message: PCBs update
Parts:
- added D112, D113: LED, LED_SMD:LED_0805_2012Metric_Pad1.15x1.40mm_HandSolder, symbol Device:LED
- added R86, R87: 290, Capacitor_SMD:C_0805_2012Metric_Pad1.18x1.45mm_HandSolder, symbol Device:R
- gave numbers to parts that had none: 36
Connections:
- net +3.3V: now also R86.1, R87.1
- net UART3RX: now also D112.1 (K)
- net UART3TX: now also D113.1 (K)
- new net: D113.2 (A), R87.2
- new net: D112.2 (A), R86.2
