File: Motor_reroute/Motor_reroute.kicad_pcb (KiCad board)
At the start: 2 copper layers, 88 x 45 mm, 36 parts, among them J11 Conn_01x03, J14 RJCSE538001, J17 874380843, J18 874380843, J2 RJCSE538001, J3 Conn_01x03, J7 Conn_01x05, J8 Conn_01x05

Commit message: added pcb updates
Parts:
- removed J7, J8: Conn_01x05, Connector_JST:JST_EH_B5B-EH-A_1x05_P2.50mm_Vertical
- added J15: RJCSE538001, RJCSE538001:AMPHENOL_RJCSE538001, F.Cu at (79.6, 73.2)
Routing:
- net /SEA_I1: track 49.6 -> 38.0 mm
- net /SEA_A1: track 50.7 -> 40.2 mm
- net /SEA_B1: track 50.0 -> 43.7 mm
- net +5V: track 180.7 -> 186.3 mm, vias 8 -> 9
- net /SEA_B0: track 23.4 -> 19.7 mm, vias 0 -> 2
- net /SEA_I0: track 18.2 -> 20.8 mm
- net /SEA_A0: track 19.8 -> 19.1 mm, vias 0 -> 2
