File: Motor_Joint_Splitter_V2/Motor_Joint_Splitter_V2_alt.kicad_sch (KiCad schematic)
At the start: 17 parts, among them J1 Conn_01x08, J2 54602-908LF, J4 26605030, J7 Conn_01x05, U1 74ACT244MTCX

Commit message: Finished the first version of the new splitter PCB.
TODO:
- Update connectors to IDCs if we can find some 5 pin and 8 pin ones.
- Add part numbers for LCSC fields.
- Generate bill of materials.
Parts:
- added R10, R11, R12, R7, R8, R9: 0Ω, PCM_JLCPCB:R_0402, symbol PCM_JLCPCB-Resistors:0402,0Ω
Connections:
- net C_A: now also U1.2 (I0); no longer U1.6 (I2)
- net C_A_Out: now also U1.18 (O0), R7.1; no longer D5.6 (A), D5.6 (K), U1.14 (O2)
- net C_B: now also U1.4 (I1); no longer U1.8 (I3)
- net C_B_Out: now also U1.16 (O1), R8.1; no longer D5.3 (A), D5.3 (K), U1.12 (O3)
- net C_I: now also U1.6 (I2); no longer U1.2 (I0)
- net C_I_Out: now also U1.14 (O2), R12.1; no longer D6.6 (A), D6.6 (K), U1.18 (O0)
- net SEA_A: now also U1.8 (I3); no longer U1.15 (I5)
- net SEA_A_Out: now also U1.12 (O3), R9.1; no longer D7.6 (A), D7.6 (K), U1.5 (O5)
- net SEA_B_Out: now also R10.1; no longer D7.3 (A), D7.3 (K)
- net SEA_I: now also U1.15 (I5); no longer U1.4 (I1)
- net SEA_I_Out: now also U1.5 (O5), R11.1; no longer D6.3 (A), D6.3 (K), U1.16 (O1)
- new net: D5.6 (A), D5.6 (K), R7.2
- new net: D6.3 (A), D6.3 (K), R11.2
- new net: D6.6 (A), D6.6 (K), R12.2
- new net: D5.3 (A), D5.3 (K), R8.2
- new net: D7.3 (A), D7.3 (K), R10.2
- new net: D7.6 (A), D7.6 (K), R9.2
