File: Motor_Joint_Splitter_V2/Motor_Joint_Splitter_V2.kicad_pcb (KiCad board)
At the start: 2 copper layers, 45 x 45 mm, 21 parts, among them J2 26605030, J7 ethernet_54602-908LF, J8 motor_connector_292206-8, J9 Conn_01x05, U2 74ACT244MTCX

Commit message: Board seems mostly complete. Need to verify parts list and gerber files are fine next.
Parts:
- C2, C4: moved to F.Cu
- moved C2 32.2 mm to (210.2, 70.6)
- moved C4 21.8 mm to (201.0, 73.2), turned to 180 degrees
- moved R17 11.7 mm to (201.4, 83.6), turned to -90 degrees
- moved D7 11.6 mm to (197.6, 82.4), turned to 0 degrees
- moved D6 10.5 mm to (203.4, 76.2), turned to -90 degrees
- moved R19 6.68 mm to (194.0, 83.6), turned to -90 degrees
- moved R13 4.90 mm to (190.8, 80.6), turned to -90 degrees
- moved D4 3.76 mm to (185.4, 87.6)
- moved U2 3.30 mm to (197.6, 77.2)
- moved D5 2.53 mm to (192.0, 76.2), turned to 90 degrees
- moved R15 2.01 mm to (204.0, 80.0)
- moved R16 1.81 mm to (206.6, 80.0)
- moved R14 1.62 mm to (188.2, 80.6), turned to -90 degrees
- moved H2 0.36 mm to (221.5, 101.5)
- moved H3 0.22 mm to (221.5, 63.5)
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Connections:
- D5 pad 6: /C_A_Out -> /C_I_Out
- D6 pad 3: /SEA_I_Out -> /SEA_B_Out
- D6 pad 6: /C_I_Out -> /SEA_A_Out
- D7 pad 3: /SEA_B_Out -> /C_A_Out
- D7 pad 6: /SEA_A_Out -> /SEA_I_Out
Routing:
- net +5V: track 1.90 -> 92.9 mm, vias 0 -> 3
- net GND: track 0.00 -> 69.9 mm, vias 0 -> 2
- net /Cos: track 0.00 -> 18.6 mm
- net /Sin: track 0.00 -> 18.2 mm
- net /C_I_Out_2: track 0.00 -> 16.6 mm
- net /SEA_B_Out_2: track 0.00 -> 12.8 mm
- net /SEA_A_Out_2: track 0.00 -> 10.5 mm
- net /C_B_Out_2: track 0.00 -> 10.2 mm
- net /SEA_I_Out_2: track 0.00 -> 8.11 mm
- net /SEA_I_Out: track 15.8 -> 9.08 mm
- net /SEA_B: track 4.78 -> 10.9 mm
- net /C_A_Out_2: track 0.00 -> 4.05 mm
- net /C_B: track 12.1 -> 14.3 mm
- net /C_A_Out: track 10.4 -> 8.23 mm
- net /C_I: track 8.16 -> 10.3 mm
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- added copper zone on B.Cu, net GND
- added copper zone on F.Cu, net GND
